File: Engine/OpenHO_Engine/OpenHO_Engine.kicad_pcb (KiCad board)
At the start: 2 copper layers, 6 x 2.5 mm, 0 parts

Commit message: SUKU engine mock up created
Parts:
- added J1: Conn_01x01, TestPoint:TestPoint_THTPad_1.0x1.0mm_Drill0.5mm, F.Cu at (146.5, 105.0)
- added J1: Conn_01x01, TestPoint:TestPoint_THTPad_1.0x1.0mm_Drill0.5mm, F.Cu at (96.5, 105.0)
- added J2: Conn_01x01, TestPoint:TestPoint_THTPad_1.0x1.0mm_Drill0.5mm, F.Cu at (150.0, 101.5)
- added J2: Conn_01x01, TestPoint:TestPoint_THTPad_1.0x1.0mm_Drill0.5mm, F.Cu at (100.0, 101.5)
- added J4: Conn_01x01, TestPoint:TestPoint_THTPad_1.0x1.0mm_Drill0.5mm, F.Cu at (153.5, 105.0)
- added J4: Conn_01x01, TestPoint:TestPoint_THTPad_1.0x1.0mm_Drill0.5mm, F.Cu at (103.5, 105.0)
Other:
- board size 6 x 2.5 mm -> 90 x 41 mm

Commit message: SUKU protopcb order for Track & Engine
Parts:
- removed the J1 at (146.5, 105.0)
- removed the J1 at (96.5, 105.0)
- removed the J2 at (150.0, 101.5)
- removed the J2 at (100.0, 101.5)
- removed the J4 at (153.5, 105.0)
- removed the J4 at (103.5, 105.0)
- added C1: CAP, suku_basics:CAP_0805, F.Cu at (157.0, 77.5)
- added C2: CAP, suku_basics:CAP_0805, F.Cu at (151.0, 77.5)
- added C3: CAP, suku_basics:CAP_0805, F.Cu at (147.5, 77.5)
- added C4: CAP, suku_basics:CAP_0805, F.Cu at (145.5, 77.5)
- added D1: LED, suku_basics:LED_0805, B.Cu at (85.0, 89.0)
- added D10: LED, suku_basics:LED_0805, B.Cu at (135.0, 89.0)
- added D11: LED, suku_basics:LED_0805, B.Cu at (140.0, 89.0)
- added D12: SCHOTTKY, Diode_SMD:D_SOD-123, B.Cu at (143.0, 86.0)
- added D13: SCHOTTKY, Diode_SMD:D_SOD-123, B.Cu at (157.0, 86.0)
- added D14: LED, suku_basics:LED_0805, B.Cu at (160.0, 89.0)
- added D15: LED, suku_basics:LED_0805, B.Cu at (165.0, 89.0)
- added D16: LED, suku_basics:LED_0805, B.Cu at (85.0, 66.0)
- added D17: LED, suku_basics:LED_0805, B.Cu at (90.0, 66.0)
- added D18: SCHOTTKY, Diode_SMD:D_SOD-123, B.Cu at (107.0, 69.0)
- added D19: SCHOTTKY, Diode_SMD:D_SOD-123, B.Cu at (93.0, 69.0)
- added D2: LED, suku_basics:LED_0805, B.Cu at (90.0, 89.0)
- added D20: LED, suku_basics:LED_0805, B.Cu at (110.0, 66.0)
- added D21: LED, suku_basics:LED_0805, B.Cu at (115.0, 66.0)
- added D22: LED, suku_basics:LED_0805, B.Cu at (120.0, 66.0)
- added D23: LED, suku_basics:LED_0805, B.Cu at (125.0, 66.0)
- added D24: LED, suku_basics:LED_0805, B.Cu at (130.0, 66.0)
- added D25: LED, suku_basics:LED_0805, B.Cu at (135.0, 66.0)
- added D26: LED, suku_basics:LED_0805, B.Cu at (140.0, 66.0)
- added D27: SCHOTTKY, Diode_SMD:D_SOD-123, B.Cu at (143.0, 69.0)
- added D28: SCHOTTKY, Diode_SMD:D_SOD-123, B.Cu at (157.0, 69.0)
- added D29: LED, suku_basics:LED_0805, B.Cu at (160.0, 66.0)
- added D3: SCHOTTKY, Diode_SMD:D_SOD-123, B.Cu at (107.0, 86.0)
- added D30: LED, suku_basics:LED_0805, B.Cu at (165.0, 66.0)
- added D4: SCHOTTKY, Diode_SMD:D_SOD-123, B.Cu at (93.0, 86.0)
- added D5: LED, suku_basics:LED_0805, B.Cu at (110.0, 89.0)
- added D6: LED, suku_basics:LED_0805, B.Cu at (115.0, 89.0)
- added D7: LED, suku_basics:LED_0805, B.Cu at (120.0, 89.0)
- added D8: LED, suku_basics:LED_0805, B.Cu at (125.0, 89.0)
- added D9: LED, suku_basics:LED_0805, B.Cu at (130.0, 89.0)
- added H1: MountingHole, suku_basics:PANEL_BREAKOUT-2x3-0.7, F.Cu at (82.5, 63.2)
- added H2: MountingHole, suku_basics:PANEL_BREAKOUT-2x3-0.7, F.Cu at (167.5, 91.8)
- added H3: MountingHole, suku_basics:PANEL_BREAKOUT-2x3-0.7, F.Cu at (167.5, 63.2)
- added H4: MountingHole, suku_basics:PANEL_BREAKOUT-2x3-0.7, F.Cu at (82.5, 91.8)
- added J1: Conn_01x01, TestPoint:TestPoint_THTPad_1.0x1.0mm_Drill0.5mm, B.Cu at (96.5, 100.0)
- added J2: Conn_01x01, TestPoint:TestPoint_THTPad_1.0x1.0mm_Drill0.5mm, B.Cu at (103.5, 100.0)
- added J3: Conn_01x01, TestPoint:TestPoint_THTPad_1.0x1.0mm_Drill0.5mm, B.Cu at (146.5, 100.0)
- added J4: Conn_01x01, TestPoint:TestPoint_THTPad_1.0x1.0mm_Drill0.5mm, B.Cu at (153.5, 100.0)
- added J5: Conn_01x01, TestPoint:TestPoint_THTPad_1.0x1.0mm_Drill0.5mm, B.Cu at (96.5, 55.0)
- added J6: Conn_01x01, TestPoint:TestPoint_THTPad_1.0x1.0mm_Drill0.5mm, B.Cu at (103.5, 55.0)
- added J7: Conn_01x01, TestPoint:TestPoint_THTPad_1.0x1.0mm_Drill0.5mm, B.Cu at (146.5, 55.0)
- added J8: Conn_01x01, TestPoint:TestPoint_THTPad_1.0x1.0mm_Drill0.5mm, B.Cu at (153.5, 55.0)
- added R1: RES, suku_basics:RES_0805, B.Cu at (85.0, 87.0)
- added R10: RES, suku_basics:RES_0805, B.Cu at (125.0, 87.0)
- added R11: RES, suku_basics:RES_0805, B.Cu at (130.0, 87.0)
- added R12: RES, suku_basics:RES_0805, B.Cu at (135.0, 87.0)
- added R13: RES, suku_basics:RES_0805, B.Cu at (140.0, 87.0)
- added R14: RES, Resistor_THT:R_Axial_DIN0309_L9.0mm_D3.2mm_P12.70mm_Horizontal, B.Cu at (143.0, 83.5)
- added R15: RES, suku_basics:RES_0805, F.Cu at (147.5, 81.0)
- added R16: RES, Resistor_THT:R_Axial_DIN0309_L9.0mm_D3.2mm_P12.70mm_Horizontal, B.Cu at (157.0, 83.5)
- added R17: RES, suku_basics:RES_0805, B.Cu at (160.0, 87.0)
- added R18: RES, suku_basics:RES_0805, B.Cu at (165.0, 87.0)
- added R19: RES, suku_basics:RES_0805, F.Cu at (149.5, 81.0)
- added R2: RES, suku_basics:RES_0805, B.Cu at (90.0, 87.0)
- added R20: RES, suku_basics:RES_0805, B.Cu at (85.0, 68.0)
- added R21: RES, suku_basics:RES_0805, B.Cu at (90.0, 68.0)
- added R22: RES, suku_basics:RES_0805, F.Cu at (145.5, 74.0)
- added R23: RES, Resistor_THT:R_Axial_DIN0309_L9.0mm_D3.2mm_P12.70mm_Horizontal, B.Cu at (93.0, 71.5)
- added R24: RES, Resistor_THT:R_Axial_DIN0309_L9.0mm_D3.2mm_P12.70mm_Horizontal, B.Cu at (107.0, 71.5)
- added R25: RES, suku_basics:RES_0805, B.Cu at (110.0, 68.0)
- added R26: RES, suku_basics:RES_0805, B.Cu at (115.0, 68.0)
- added R27: RES, suku_basics:RES_0805, B.Cu at (120.0, 68.0)
- added R28: RES, suku_basics:RES_0805, B.Cu at (125.0, 68.0)
- added R29: RES, suku_basics:RES_0805, B.Cu at (130.0, 68.0)
- added R3: RES, suku_basics:RES_0805, F.Cu at (145.5, 81.0)
- added R30: RES, suku_basics:RES_0805, B.Cu at (135.0, 68.0)
- added R31: RES, suku_basics:RES_0805, B.Cu at (140.0, 68.0)
- added R32: RES, Resistor_THT:R_Axial_DIN0309_L9.0mm_D3.2mm_P12.70mm_Horizontal, B.Cu at (143.0, 71.5)
- added R33: RES, suku_basics:RES_0805, F.Cu at (147.5, 74.0)
- added R34: RES, Resistor_THT:R_Axial_DIN0309_L9.0mm_D3.2mm_P12.70mm_Horizontal, B.Cu at (157.0, 71.5)
- added R35: RES, suku_basics:RES_0805, B.Cu at (160.0, 68.0)
- added R36: RES, suku_basics:RES_0805, B.Cu at (165.0, 68.0)
- added R4: RES, Resistor_THT:R_Axial_DIN0309_L9.0mm_D3.2mm_P12.70mm_Horizontal, B.Cu at (93.0, 83.5)
- added R5: RES, Resistor_THT:R_Axial_DIN0309_L9.0mm_D3.2mm_P12.70mm_Horizontal, B.Cu at (107.0, 83.5)
- added R6: RES, suku_basics:RES_0805, B.Cu at (110.0, 87.0)
- added R7: RES, suku_basics:RES_0805, B.Cu at (115.0, 87.0)
- added R8: RES, suku_basics:RES_0805, F.Cu at (159.0, 77.5)
- added R9: RES, suku_basics:RES_0805, B.Cu at (120.0, 87.0)
- added TP1: TestPoint_2Pole, TestPoint:TestPoint_2Pads_Pitch5.08mm_Drill1.3mm, F.Cu at (143.0, 80.0)
- added U1: U_REGULATOR_SOT23-5, suku_basics:SOT-23-5, F.Cu at (154.0, 77.5)
Routing:
- net -VDC: track 0.00 -> 169.2 mm, vias 0 -> 7
- net +VDC: track 0.00 -> 118.9 mm, vias 0 -> 5
- net Net-(D3-Pad2): track 0.00 -> 56.1 mm
- net Net-(D18-Pad2): track 0.00 -> 56.1 mm
- net Net-(J3-Pad1): track 0.00 -> 21.8 mm
- net Net-(J1-Pad1): track 0.00 -> 21.8 mm
- net Net-(J7-Pad1): track 0.00 -> 21.8 mm
- net Net-(J5-Pad1): track 0.00 -> 21.8 mm
- net Net-(D12-Pad2): track 0.00 -> 17.2 mm
- net Net-(D27-Pad2): track 0.00 -> 17.2 mm
- net -VSW: track 0.00 -> 8.41 mm
- net +VSW: track 0.00 -> 8.41 mm
- net VBUS: track 0.00 -> 7.25 mm
- net Net-(D9-Pad2): track 0.00 -> 2.00 mm
- net Net-(D8-Pad2): track 0.00 -> 2.00 mm
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- added copper zone on F.Cu, net +3V3
- added copper zone on B.Cu, net GND
Other:
- board size 90 x 41 mm -> 90 x 47 mm
- rule solder_mask_min_width: 0.25 -> 0.05
