File: Engine/OpenHO_Engine/OpenHO_Engine.sch (KiCad schematic (older format))
At the start: 3 parts

Commit message: SUKU engine mock up created
Parts:
- added D1, D2, D3, D4: SCHOTTKY, symbol agro-symbol:SCHOTTKY
- added D5, D6, D7: LED, suku_basics:LED_0805, symbol suku_basics:LED
- added J4, J5, J6: Conn_01x01, TestPoint:TestPoint_THTPad_1.0x1.0mm_Drill0.5mm, symbol Connector_Generic:Conn_01x01
- added R1, R2, R3: RES, suku_basics:RES_0805, symbol suku_basics:RES
- added U1: U_REGULATOR_SOT23-5, suku_basics:SOT-23-5, symbol suku_basics:U_REGULATOR_SOT23-5
- J1, J2, J3: renamed from J?; footprint TestPoint:TestPoint_THTPad_2.5x2.5mm_Drill1.2mm -> TestPoint:TestPoint_THTPad_1.0x1.0mm_Drill0.5mm
Connections:
- net labels added: +3V3, +VDC, -VDC, GND, VBUS
- wire segments 4 -> 43
Other:
- moved on the sheet: J1, J2, J3

Commit message: SUKU protopcb order for Track & Engine
Parts:
- removed D1, D2, D3, D4: SCHOTTKY, symbol agro-symbol:SCHOTTKY
- removed D5, D6, D7: LED, suku_basics:LED_0805, symbol suku_basics:LED
- removed J1, J2, J3, J4, J5, J6: Conn_01x01, TestPoint:TestPoint_THTPad_1.0x1.0mm_Drill0.5mm, symbol Connector_Generic:Conn_01x01
- removed R1, R2, R3: RES, suku_basics:RES_0805, symbol suku_basics:RES
- added C1, C2, C3, C4: CAP, suku_basics:CAP_0805, symbol suku_basics:CAP
- added R19, R8: RES, suku_basics:RES_0805, symbol suku_basics:RES
- added TP1: TestPoint_2Pole, TestPoint:TestPoint_2Pads_Pitch5.08mm_Drill1.3mm, symbol Connector:TestPoint_2Pole
Connections:
- net +3V3: now also C2.1
- net +VDC: now also R8.2
- net -VDC: now also R19.2
- net GND: now also C1.2, C2.2, R19.1
- net VBUS: now also C1.1, R8.1
- new net +VSW: C3.1, C4.1, TP1.1
- new net -VSW: C3.2, C4.2, TP1.2
Other:
- moved on the sheet: U1
