File: Tracks/S174/S174.kicad_pcb (KiCad board)
At the start: 2 copper layers, 174 x 30 mm, 48 parts, among them J1 Conn_01x02, J2 Conn_01x04, J3 Conn_01x02, J4 Conn_01x02, J5 Conn_01x04, J6 Conn_01x02, U1 A4953_LJ, U2 ATmega328PB-AU

Commit message: SUKU protopcb order for Track & Engine
Parts:
- removed F1, F2: POLY, suku_basics:POLY_0805
- removed R1, R2: RES, suku_basics:RES_0805
- removed TP11: TestPoint, suku_basics:HO_tie
- removed U1: A4953_LJ, Package_SO:SOIC-8-1EP_3.9x4.9mm_P1.27mm_EP2.41x3.3mm
- removed U2: ATmega328PB-AU, Package_QFP:TQFP-32_7x7mm_P0.8mm
- added TP10: TestPoint, suku_basics:HO_tie, F.Cu at (268.0, 108.5)
- added TP2: TestPoint, suku_basics:HO_tie, F.Cu at (106.0, 108.5)
- added TP4: TestPoint, suku_basics:HO_tie, F.Cu at (146.5, 108.5)
- added TP6: TestPoint, suku_basics:HO_tie, F.Cu at (187.0, 108.5)
- added TP8: TestPoint, suku_basics:HO_tie, F.Cu at (227.5, 108.5)
Routing:
- net Net-(J2-Pad3): track 0.00 -> 172.0 mm
- net Net-(J2-Pad2): track 0.00 -> 172.0 mm
- net GND: track 0.00 -> 172.0 mm
- net +5V: track 0.00 -> 172.0 mm
- net -VSW: track 0.00 -> 162.0 mm
- net +VSW: track 0.00 -> 162.0 mm
