File: Tracks/S174/S174.sch (KiCad schematic (older format))
At the start: 24 parts, among them J1 Conn_01x02, J2 Conn_01x04, J3 Conn_01x02, J4 Conn_01x02, J5 Conn_01x04, J6 Conn_01x02, U1 A4953_LJ, U2 ATmega328PB-AU

Commit message: SUKU protopcb order for Track & Engine
Parts:
- removed F1, F2: POLY, suku_basics:POLY_0805, symbol suku_basics:POLY
- removed R1, R2: RES, suku_basics:RES_0805, symbol suku_basics:RES
- removed TP11: TestPoint, suku_basics:HO_tie, symbol Connector:TestPoint
- removed TP12: TestPoint, symbol Connector:TestPoint
- removed U1: A4953_LJ, Package_SO:SOIC-8-1EP_3.9x4.9mm_P1.27mm_EP2.41x3.3mm, symbol Driver_Motor:A4953_LJ
- removed U2: ATmega328PB-AU, Package_QFP:TQFP-32_7x7mm_P0.8mm, symbol MCU_Microchip_ATmega:ATmega328PB-AU
- TP10, TP2, TP4, TP6, TP8: footprint (none) -> suku_basics:HO_tie
Changed lines of the file:
@@
 EESchema Schematic File Version 4
-LIBS:HO_Turnout_No4-cache
+LIBS:S174-cache
 EELAYER 29 0
 EELAYER END
@@
 $EndComp
 $Comp
-L Connector:TestPoint TP11
-U 1 1 5E18A009
-P 3100 2700
-F 0 "TP11" H 3158 2818 50  0001 L CNN
-F 1 "TestPoint" H 3158 2727 50  0001 L CNN
-F 2 "suku_basics:HO_tie" H 3300 2700 50  0001 C CNN
-F 3 "~" H 3300 2700 50  0001 C CNN
-	1    3100 2700
-	1    0    0    -1
-$EndComp
-$Comp
 L Connector:TestPoint TP2
 U 1 1 5E18BBDE
@@
 F 0 "TP2" H 2158 4618 50  0001 L CNN
 F 1 "TestPoint" H 2158 4527 50  0001 L CNN
-F 2 "" H 2300 4500 50  0001 C CNN
+F 2 "suku_basics:HO_tie" H 2300 4500 50  0001 C CNN
 F 3 "~" H 2300 4500 50  0001 C CNN
 	1    2100 4500
@@
 F 0 "TP4" H 2358 4618 50  0001 L CNN
 F 1 "TestPoint" H 2358 4527 50  0001 L CNN
-F 2 "" H 2500 4500 50  0001 C CNN
+F 2 "suku_basics:HO_tie" H 2500 4500 50  0001 C CNN
 F 3 "~" H 2500 4500 50  0001 C CNN
 	1    2300 4500
@@
 F 0 "TP6" H 2558 4618 50  0001 L CNN
 F 1 "TestPoint" H 2558 4527 50  0001 L CNN
-F 2 "" H 2700 4500 50  0001 C CNN
+F 2 "suku_basics:HO_tie" H 2700 4500 50  0001 C CNN
 F 3 "~" H 2700 4500 50  0001 C CNN
 	1    2500 4500
@@
 F 0 "TP8" H 2758 4618 50  0001 L CNN
 F 1 "TestPoint" H 2758 4527 50  0001 L CNN
-F 2 "" H 2900 4500 50  0001 C CNN
+F 2 "suku_basics:HO_tie" H 2900 4500 50  0001 C CNN
 F 3 "~" H 2900 4500 50  0001 C CNN
 	1    2700 4500
@@
 F 0 "TP10" H 2958 4618 50  0001 L CNN
 F 1 "TestPoint" H 2958 4527 50  0001 L CNN
-F 2 "" H 3100 4500 50  0001 C CNN
+F 2 "suku_basics:HO_tie" H 3100 4500 50  0001 C CNN
 F 3 "~" H 3100 4500 50  0001 C CNN
 	1    2900 4500
 	1    0    0    -1
 $EndComp
-$Comp
-L Connector:TestPoint TP12
-U 1 1 5E18BBFC
-P 3100 4500
-F 0 "TP12" H 3158 4618 50  0001 L CNN
-F 1 "TestPoint" H 3158 4527 50  0001 L CNN
-F 2 "" H 3300 4500 50  0001 C CNN
-F 3 "~" H 3300 4500 50  0001 C CNN
-	1    3100 4500
-	1    0    0    -1
-$EndComp
 Wire Wire Line
 	2100 2700 2100 2800
 Wire Wire Line
 	2100 2800 2300 2800
-Wire Wire Line
-	3100 2800 3100 2700
 Wire Wire Line
 	2900 2700 2900 2800
 Connection ~ 2900 2800
 Wire Wire Line
-	2900 2800 3100 2800
-Wire Wire Line
 	2700 2700 2700 2800
 Connection ~ 2700 2800
@@
 	2100 4600 2300 4600
 Wire Wire Line
-	3100 4600 3100 4500
-Wire Wire Line
 	2900 4500 2900 4600
 Connection ~ 2900 4600
 Wire Wire Line
-	2900 4600 3100 4600
-Wire Wire Line
 	2700 4500 2700 4600
 Connection ~ 2700 4600
@@
 Wire Wire Line
 	2300 4600 2500 4600
-$Comp
-L suku_basics:RES R1
-U 1 1 5E190E43
-P 10000 3300
-F 0 "R1" H 10059 3346 50  0000 L CNN
-F 1 "RES" H 10059 3255 50  0000 L CNN
-F 2 "suku_basics:RES_0805" H 10000 3300 50  0001 C CNN
-F 3 "~" H 10000 3300 50  0001 C CNN
-	1    10000 3300
-	1    0    0    -1
-$EndComp
-$Comp
-L suku_basics:RES R2
-U 1 1 5E191434
-P 10400 3300
-F 0 "R2" H 10459 3346 50  0000 L CNN
-F 1 "RES" H 10459 3255 50  0000 L CNN
-F 2 "suku_basics:RES_0805" H 10400 3300 50  0001 C CNN
-F 3 "~" H 10400 3300 50  0001 C CNN
-	1    10400 3300
-	1    0    0    -1
-$EndComp
-$Comp
-L Driver_Motor:A4953_LJ U1
-U 1 1 5E1949B1
-P 5000 3300
-F 0 "U1" H 5000 3881 50  0000 C CNN
-F 1 "A4953_LJ" H 5000 3790 50  0000 C CNN
-F 2 "Package_SO:SOIC-8-1EP_3.9x4.9mm_P1.27mm_EP2.41x3.3mm" H 5000 2750 50  0001 C CNN
-F 3 "www.allegromicro.com/~/media/Files/Datasheets/A4952-3-Datasheet.ashx?la=en" H 4700 3650 50  0001 C CNN
-	1    5000 3300
-	1    0    0    -1
-$EndComp
-$Comp
-L MCU_Microchip_ATmega:ATmega328PB-AU U2
-U 1 1 5E19835F
-P 8700 4200
-F 0 "U2" H 8700 2611 50  0000 C CNN
-F 1 "ATmega328PB-AU" H 8700 2520 50  0000 C CNN
-F 2 "Package_QFP:TQFP-32_7x7mm_P0.8mm" H 8700 4200 50  0001 C CIN
-F 3 "http://ww1.microchip.com/downloads/en/DeviceDoc/40001906C.pdf" H 8700 4200 50  0001 C CNN
-	1    8700 4200
-	1    0    0    -1
-$EndComp
 $Comp
 L power:+5V #PWR0103
@@
 Wire Wire Line
 	2400 3400 3000 3400
-$Comp
-L power:GND #PWR0105
-U 1 1 5E1A3D38
-P 8700 6100
-F 0 "#PWR0105" H 8700 5850 50  0001 C CNN
-F 1 "GND" H 8705 5927 50  0000 C CNN
-F 2 "" H 8700 6100 50  0001 C CNN
-F 3 "" H 8700 6100 50  0001 C CNN
-	1    8700 6100
-	1    0    0    -1
-$EndComp
-$Comp
-L power:+5V #PWR0106
-U 1 1 5E1A4626
-P 8700 2500
-F 0 "#PWR0106" H 8700 2350 50  0001 C CNN
-F 1 "+5V" H 8715 2673 50  0000 C CNN
-F 2 "" H 8700 2500 50  0001 C CNN
-F 3 "" H 8700 2500 50  0001 C CNN
-	1    8700 2500
-	1    0    0    -1
-$EndComp
-Wire Wire Line
-	8700 2500 8700 2700
-$Comp
-L power:GND #PWR0107
-U 1 1 5E1A549A
-P 5000 3800
-F 0 "#PWR0107" H 5000 3550 50  0001 C CNN
-F 1 "GND" H 5005 3627 50  0000 C CNN
-F 2 "" H 5000 3800 50  0001 C CNN
-F 3 "" H 5000 3800 50  0001 C CNN
-	1    5000 3800
-	1    0    0    -1
-$EndComp
-Wire Wire Line
-	5000 3800 5000 3700
 $Sheet
 S 4000 -6000 1000 300
@@
 Wire Wire Line
 	3600 2700 3600 2800
-Wire Wire Line
-	3600 2800 3100 2800
-Connection ~ 3100 2800
 $Comp
 L power:-VSW #PWR0109
@@
 	3600 4500 3600 4600
 Wire Wire Line
-	3600 4600 3100 4600
-Connection ~ 3100 4600
-$Comp
-L power:+VSW #PWR0110
-U 1 1 5E22BE95
-P 6400 3000
-F 0 "#PWR0110" H 6400 2850 50  0001 C CNN
-F 1 "+VSW" H 6415 3173 50  0000 C CNN
-F 2 "" H 6400 3000 50  0001 C CNN
-F 3 "" H 6400 3000 50  0001 C CNN
-	1    6400 3000
-	1    0    0    -1
-$EndComp
-Wire Wire Line
-	6400 3000 6400 3100
-$Comp
-L power:-VSW #PWR0111
-U 1 1 5E22BE9D
-P 6600 3100
-F 0 "#PWR0111" H 6600 3200 50  0001 C CNN
-F 1 "-VSW" H 6615 3273 50  0000 C CNN
-F 2 "" H 6600 3100 50  0001 C CNN
-F 3 "" H 6600 3100 50  0001 C CNN
-	1    6600 3100
-	1    0    0    -1
-$EndComp
-Wire Wire Line
-	6600 3100 6600 3200
-$Comp
-L suku_basics:POLY F1
-U 1 1 5E2321CC
-P 5700 3100
-F 0 "F1" V 5495 3100 50  0000 C CNN
-F 1 "POLY" V 5586 3100 50  0000 C CNN
-F 2 "suku_basics:POLY_0805" H 5750 2900 50  0001 L CNN
-F 3 "~" H 5700 3100 50  0001 C CNN
-	1    5700 3100
-	0    1    1    0
-$EndComp
-$Comp
-L suku_basics:POLY F2
-U 1 1 5E232B71
-P 5700 3200
-F 0 "F2" V 5495 3200 50  0000 C CNN
-F 1 "POLY" V 5586 3200 50  0000 C CNN
-F 2 "suku_basics:POLY_0805" H 5750 3000 50  0001 L CNN
-F 3 "~" H 5700 3200 50  0001 C CNN
-	1    5700 3200
-	0    1    1    0
-$EndComp
-Wire Wire Line
-	5800 3100 6400 3100
-Wire Wire Line
-	5800 3200 6600 3200
-Wire Wire Line
-	5600 3100 5400 3100
-Wire Wire Line
-	5400 3200 5600 3200
+	2900 4600 3600 4600
+Wire Wire Line
+	2900 2800 3600 2800
 $EndSCHEMATC
